Commit message: minor_changes

File: src/urdf/robot.urdf (robot description, URDF)
Before this commit: robot six_dof_robot, 8 links, 7 joints
Links:
- removed link gripper_base
- removed link link1
- removed link link2
- removed link link3
- removed link link4
- removed link link5
- removed link link6
- added link Gripper_1, mass 0.137742996071251; collision mesh filename=file:///home/deepak/6_dof/meshes/Gripper_1.STL; visual mesh filename=file:///home/deepak/6_dof/meshes/Gripper_1.STL
- added link Gripper_2, mass 0.153524806277575; collision mesh filename=file:///home/deepak/6_dof/meshes/Gripper_2.STL; visual mesh filename=file:///home/deepak/6_dof/meshes/Gripper_2.STL
- added link Link_1, mass 2.19576081627391; collision mesh filename=file:///home/deepak/6_dof/meshes/Link_1.STL; visual mesh filename=file:///home/deepak/6_dof/meshes/Link_1.STL
- added link Link_2, mass 0.696616277349387; collision mesh filename=file:///home/deepak/6_dof/meshes/Link_2.STL; visual mesh filename=file:///home/deepak/6_dof/meshes/Link_2.STL
- added link Link_3, mass 0.504770554183686; collision mesh filename=file:///home/deepak/6_dof/meshes/Link_3.STL; visual mesh filename=file:///home/deepak/6_dof/meshes/Link_3.STL
- added link Link_4, mass 0.739327182415655; collision mesh filename=file:///home/deepak/6_dof/meshes/Link_4.STL; visual mesh filename=file:///home/deepak/6_dof/meshes/Link_4.STL
- added link Link_5, mass 0.0763957117756357; collision mesh filename=file:///home/deepak/6_dof/meshes/Link_5.STL; visual mesh filename=file:///home/deepak/6_dof/meshes/Link_5.STL
- added link Link_6, mass 0.252745339929401; collision mesh filename=file:///home/deepak/6_dof/meshes/Link_6.STL; visual mesh filename=file:///home/deepak/6_dof/meshes/Link_6.STL
- added link camera_link_base_left, mass 1e-5; collision box size=0.025 0.025 0.025; visual box size=0.025 0.025 0.025
- added link camera_link_base_right, mass 1e-5; collision box size=0.025 0.025 0.025; visual box size=0.025 0.025 0.025
- added link camera_link_gripper_left, mass 1e-5; collision box size=0.025 0.025 0.025; visual box size=0.025 0.025 0.025
- added link camera_link_gripper_right, mass 1e-5; collision box size=0.025 0.025 0.025; visual box size=0.025 0.025 0.025
- added link camera_link_optical_base_left
- added link camera_link_optical_base_right
- added link camera_link_optical_gripper_1
- added link camera_link_optical_gripper_2
- added link world
- link base_link: mass 10.0 -> 0.77116648882986; geometry collision mesh filename=file:///home/deepak/6_dof/meshes/base_link.STL; visual mesh filename=file:///home/deepak/6_dof/meshes/base_link.STL
Joints:
- removed joint gripper_base_joint
- removed joint joint1
- removed joint joint2
- removed joint joint3
- removed joint joint4
- removed joint joint5
- removed joint joint6
- added joint Finger_1: type prismatic, parent Link_6, child Gripper_1, origin xyz=0.00534999999999963 -0.0390954035350414 0.0487946645392847 rpy=1.5707963267949 0 1.5707963267949, axis 0 0 -1, limit lower=0 upper=0.0355 effort=100 velocity=10
- added joint Finger_2: type prismatic, parent Link_6, child Gripper_2, origin xyz=0.00534999999999963 -0.0390954035350414 0.0487946645392847 rpy=1.5707963267949 0 1.5707963267949, axis 0 0 -1, limit lower=-0.0355 upper=0 effort=100 velocity=10
- added joint Joint_1: type revolute, parent base_link, child Link_1, origin xyz=0 0 0.073 rpy=0 0 0, axis 0 0 1, limit lower=-3.17 upper=3.17 effort=50 velocity=5
- added joint Joint_2: type revolute, parent Link_1, child Link_2, origin xyz=-0.0299999999999999 0.114999999999999 0.0450000000000004 rpy=1.5707963267949 0 1.5707963267949, axis 0 0 -1, limit lower=-1.570 upper=1.57 effort=50 velocity=5
- added joint Joint_3: type revolute, parent Link_2, child Link_3, origin xyz=0 0.45 0.0301042347134805 rpy=0 0 0, axis 0 0 -1, limit lower=-1.00 upper=1.00 effort=50 velocity=5
- added joint Joint_4: type revolute, parent Link_3, child Link_4, origin xyz=0.0424999999995649 0.0399572355492206 0.000401106428108807 rpy=0 1.5707963267949 0, axis 0 0 1, limit lower=-3.17 upper=3.17 effort=50 velocity=5
- added joint Joint_5: type revolute, parent Link_4, child Link_5, origin xyz=-0.00649999999995384 0 -0.383499999999573 rpy=0 1.5707963267949 0, axis 0 0 1, limit lower=-0.065 upper=3.17 effort=50 velocity=5
- added joint Joint_6: type revolute, parent Link_5, child Link_6, origin xyz=0 -0.0199999999999119 0.00650441096988074 rpy=1.5707963267949 -1.5707963267949 0, axis 0 0 1, limit lower=-3.17 upper=3.17 effort=50 velocity=5
- added joint camera_base_joint_right: type fixed, parent Link_1, child camera_link_base_right, origin xyz=-0.12 -0.15 0.1 rpy=0 0 -1.57, axis 0 1 0
- added joint camera_joint_base_left: type fixed, parent Link_1, child camera_link_base_left, origin xyz=0.12 -0.15 0.02 rpy=0 0 -1.57, axis 0 1 0
- added joint camera_joint_gripper_1: type fixed, parent Link_6, child camera_link_gripper_left, origin xyz=-0.08 -0.095 0.012 rpy=0 -1.57 1.57, axis 0 1 0
- added joint camera_joint_gripper_2: type fixed, parent Link_6, child camera_link_gripper_right, origin xyz=0.08 -0.095 0.012 rpy=0 -1.57 1.57, axis 0 1 0
- added joint camera_optical_joint_base_left: type fixed, parent camera_link_base_left, child camera_link_optical_base_left, origin xyz=0 0 0 rpy=-1.5707963 0 -1.5707963
- added joint camera_optical_joint_base_right: type fixed, parent camera_link_base_right, child camera_link_optical_base_right, origin xyz=0 0 0 rpy=-1.5707963 0 -1.5707963
- added joint camera_optical_joint_gripper_1: type fixed, parent camera_link_gripper_left, child camera_link_optical_gripper_1, origin xyz=0 0 0 rpy=-1.5707963 0 -1.5707963
- added joint camera_optical_joint_gripper_2: type fixed, parent camera_link_gripper_right, child camera_link_optical_gripper_2, origin xyz=0 0 0 rpy=-1.5707963 0 -1.5707963
- added joint world_joint: type fixed, parent world, child base_link, origin xyz=0 0 0.0 rpy=0 0 0
